File: devices/rpi-uHAT/rpi-uHAT.kicad_sch (KiCad schematic)
At the start: 31 parts, among them J1 GPIO, J2 JST PH, J3 JST SH, J6 PC FAN HEADER, J7 PC FAN HEADER, U1 CAT24C256, U2 AP2112K-3.3, U3 EMC2101-x-ACZL, U4 TCA9406DC, U5 TPS61170DRV

Commit message: !fixup
Parts:
- removed C7: 10u, Capacitor_SMD:C_0805_2012Metric, symbol Device:C
- removed C8: 22u, Capacitor_SMD:C_1210_3225Metric, symbol Device:C
- removed C9: 22n, Capacitor_SMD:C_0805_2012Metric, symbol Device:C
- removed D1: SS14, Diode_SMD:D_SMA, symbol Diode:SS14
- removed J7: PC FAN HEADER, Connector:FanPinHeader_1x04_P2.54mm_Vertical, symbol Connector_Generic:Conn_01x04
- removed L1: 22u, Inductor_SMD:L_Wuerth_MAPI-4020, symbol Device:L
- removed R7: 9.76k, Resistor_SMD:R_0603_1608Metric, symbol Device:R
- removed R8: 92k, Resistor_SMD:R_0603_1608Metric, symbol Device:R
- removed R9: 10.5k, Resistor_SMD:R_0603_1608Metric, symbol Device:R
- removed U5: TPS61170DRV, Package_SON:WSON-6-1EP_2x2mm_P0.65mm_EP1x1.6mm, symbol Regulator_Switching:TPS61040DRV
- C2, C3: footprint Capacitor_SMD:C_0603_1608Metric -> Capacitor_SMD:C_0805_2012Metric
Connections:
- net +5V is gone; now on net +5V_RPI: C3.1, J1.1 (Pin_1), J1.3 (Pin_3), U2.1 (VIN), U2.3 (EN)
- net +3V3: now also J2.MP (MountPin), J3.MP (MountPin)
- net GND: no longer J2.MP (MountPin), J3.MP (MountPin)
- net +12V renamed +5V_RPI
- no-connect marks 6 -> 5
Other:
- note removed: "12V@200mA Boost Converter"
- moved on the sheet: C4, J3, J6, R5, R6, U3

Commit message: [rpi-uHAT] Adds MPN for all parts.
Parts:
- C1, C4, C5, C6: MPN (none) -> CL10B104KB8NNWC
- C2, C3: MPN (none) -> CL21B105KAFNNNE
- J1: MPN (none) -> HLE-120-02-F-DV-BE
- J2: MPN (none) -> S4B-PH-SM4-TB
- J3: MPN (none) -> SM04B-SRSS-TB
- R1, R2: MPN (none) -> RC0603FR-073K9L
- R3, R4, R5, R6: MPN (none) -> RC0603FR-0710KL
- U1: MPN (none) -> CAT24C256
- U2: MPN (none) -> AP2112K-3.3
- U3: MPN (none) -> EMC2101-R-ACZL-TR
- U4: MPN (none) -> TCA9406DC
Connections:
- net GPIO4/GPCLK0 is gone; now on net EN: J1.8 (Pin_8)
- net EN: now reaches U4.6 (OE)
Other:
- moved on the sheet: C4, J3, J6, R5, R6, U3
