File: devices/rpi-uHAT/rpi-uHAT.kicad_sch (KiCad schematic)
At the start: 21 parts, among them J1 GPIO, J2 JST PH, J3 JST SH, J6 PC FAN HEADER, U1 CAT24C256, U2 AP2112K-3.3, U3 EMC2101-x-ACZL, U4 TCA9406DC

Commit message: Finsihes version A.0 of the BLE sensor
Parts:
- added C10: 100u, Capacitor_SMD:C_1206_3216Metric, symbol Device:C_Small
- added C7: 100n, Capacitor_SMD:C_0603_1608Metric, symbol Device:C_Small
- added C8: 33n, Capacitor_SMD:C_0603_1608Metric, symbol Device:C_Small
- added C9: 4u7, Capacitor_SMD:C_0805_2012Metric, symbol Device:C_Small
- added Q1: MMBT3904, Package_TO_SOT_SMD:SOT-23, symbol Transistor_BJT:MMBT3904
- added Q2: DMG2305UX, Package_TO_SOT_SMD:SOT-23, symbol Transistor_FET:DMG2301L
- added R7: 100k, Resistor_SMD:R_0603_1608Metric, symbol Device:R_Small
- added R8: 500m, Resistor_SMD:R_0603_1608Metric, symbol Device:R_Small
- J2: footprint custom:JST_PH_S4B-PH-SM4-TB_1x04-1MP_P2.00mm_Horizontal -> Connector_JST:JST_PH_B5B-PH-SM4-TB_1x05-1MP_P2.00mm_Vertical; symbol Connector_Generic_MountingPin:Conn_01x04_MountingPin -> Connector_Generic_MountingPin:Conn_01x05_MountingPin
- J3: footprint Connector_JST:JST_SH_SM04B-SRSS-TB_1x04-1MP_P1.00mm_Horizontal -> Connector_JST:JST_SH_BM04B-SRSS-TB_1x04-1MP_P1.00mm_Vertical
- R5: now not fitted
- U3: value EMC2101-x-ACZL -> EMC2101-ACZL; MPN EMC2101-R-ACZL-TR -> EMC2101-ACZL-TR
Connections:
- net +3V3: now also J2.3 (Pin_3); no longer J2.2 (Pin_2), J3.MP (MountPin)
- net +5V_RPI: now also J2.2 (Pin_2), C7.1, Q2.2 (S); no longer J6.2 (Pin_2)
- net GND: now also C9.2, R7.2, R8.2
- net SCL: now also J2.5 (Pin_5); no longer J2.4 (Pin_4)
- net SDA: now also J2.4 (Pin_4); no longer J2.3 (Pin_3)
- net DP: now reaches U3.2 (DP)
- net DP: now also Q1.1 (B), Q1.3 (C)
- net DN: now reaches U3.3 (DN)
- net DN: now also Q1.2 (E)
- new net: C10.2, R8.1
- new net +5V_FAN: C10.1, C8.1, C9.1, J6.2 (Pin_2), Q2.3 (D)
- new net SS_G: C7.2, C8.2, Q2.1 (G), R7.1
- no-connect marks 5 -> 4

Commit message: Tweeks on RPI board
Parts:
- J1: footprint custom:Samtec_HLE-120-02-xxx-DV-BE_2x20_P2.54mm_Horizontal -> Connector_PinSocket_2.54mm:PinSocket_2x20_P2.54mm_Vertical
- J2: MPN S4B-PH-SM4-TB -> B5B-PH-SM4-TB
- J3: MPN SM04B-SRSS-TB -> BM04B-SRSS-TB
Connections:
- net +3V3_RPI: now also J1.1 (Pin_1), J1.17 (Pin_17); no longer J1.18 (Pin_18), J1.2 (Pin_2)
- net +5V_RPI: now also J1.2 (Pin_2), J1.4 (Pin_4); no longer J1.1 (Pin_1), J1.3 (Pin_3)
- net EN: now also J1.7 (Pin_7); no longer J1.8 (Pin_8)
- net GND: now also J1.14 (Pin_14), J1.20 (Pin_20), J1.25 (Pin_25), J1.30 (Pin_30), J1.34 (Pin_34), J1.39 (Pin_39), J1.6 (Pin_6), J1.9 (Pin_9); no longer J1.10 (Pin_10), J1.13 (Pin_13), J1.19 (Pin_19), J1.26 (Pin_26), J1.29 (Pin_29), J1.33 (Pin_33), J1.40 (Pin_40), J1.5 (Pin_5)
- net GPIO10/SPI0.MOSI: now also J1.19 (Pin_19); no longer J1.20 (Pin_20)
- net GPIO11/SPI0.SCLK: now also J1.23 (Pin_23); no longer J1.24 (Pin_24)
- net GPIO12/PWM0: now also J1.32 (Pin_32); no longer J1.31 (Pin_31)
- net GPIO13/PWM1: now also J1.33 (Pin_33); no longer J1.34 (Pin_34)
- net GPIO14/TXD0: now also J1.8 (Pin_8); no longer J1.7 (Pin_7)
- net GPIO15/RXD0: now also J1.10 (Pin_10); no longer J1.9 (Pin_9)
- net GPIO16: now also J1.36 (Pin_36); no longer J1.35 (Pin_35)
- net GPIO17: now also J1.11 (Pin_11); no longer J1.12 (Pin_12)
- net GPIO18/PCM.CLK: now also J1.12 (Pin_12); no longer J1.11 (Pin_11)
- net GPIO19/PCM.FS: now also J1.35 (Pin_35); no longer J1.36 (Pin_36)
- net GPIO20/PCM.DIN: now also J1.38 (Pin_38); no longer J1.37 (Pin_37)
- net GPIO21/PCM.DOUT: now also J1.40 (Pin_40); no longer J1.39 (Pin_39)
- net GPIO22: now also J1.15 (Pin_15); no longer J1.16 (Pin_16)
- net GPIO23: now also J1.16 (Pin_16); no longer J1.15 (Pin_15)
- net GPIO24: now also J1.18 (Pin_18); no longer J1.17 (Pin_17)
- net GPIO25: now also J1.22 (Pin_22); no longer J1.21 (Pin_21)
- net GPIO26: now also J1.37 (Pin_37); no longer J1.38 (Pin_38)
- net GPIO27: now also J1.13 (Pin_13); no longer J1.14 (Pin_14)
- net GPIO2/SDA1: now also J1.3 (Pin_3); no longer J1.4 (Pin_4)
- net GPIO3/SCL1: now also J1.5 (Pin_5); no longer J1.6 (Pin_6)
- net GPIO5: now also J1.29 (Pin_29); no longer J1.30 (Pin_30)
- net GPIO6: now also J1.31 (Pin_31); no longer J1.32 (Pin_32)
- net GPIO7/SPI0.CE1: now also J1.26 (Pin_26); no longer J1.25 (Pin_25)
- net GPIO8/SPI0.CE0: now also J1.24 (Pin_24); no longer J1.23 (Pin_23)
- net GPIO9/SPI0.MISO: now also J1.21 (Pin_21); no longer J1.22 (Pin_22)
- net ID_SCL: now also J1.28 (Pin_28); no longer J1.27 (Pin_27)
- net ID_SDA: now also J1.27 (Pin_27); no longer J1.28 (Pin_28)
- net WP: now reaches JP1.1 (A), U1.7 (WP)
Changed lines of the file:
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@@
 	(wire
 		(pts
-			(xy 60.96 33.02) (xy 60.96 43.18)
+			(xy 60.96 68.58) (xy 60.96 80.01)
 		)
 		(stroke
@@
 	(wire
 		(pts
-			(xy 60.96 50.8) (xy 60.96 63.5)
+			(xy 58.42 35.56) (xy 85.09 35.56)
 		)
 		(stroke
@@
 	(wire
 		(pts
-			(xy 58.42 35.56) (xy 85.09 35.56)
+			(xy 43.18 38.1) (xy 43.18 58.42)
 		)
 		(stroke
@@
 	(wire
 		(pts
-			(xy 43.18 38.1) (xy 43.18 58.42)
+			(xy 60.96 33.02) (xy 60.96 43.18)
 		)
 		(stroke
@@
 	(wire
 		(pts
+			(xy 60.96 43.18) (xy 60.96 50.8)
+		)
+		(stroke
+			(width 0)
+			(type solid)
+		)
+	)
+	(wire
+		(pts
 			(xy 43.18 38.1) (xy 45.72 38.1)
 		)
@@
 	(wire
 		(pts
-			(xy 60.96 43.18) (xy 60.96 50.8)
-		)
-		(stroke
-			(width 0)
-			(type solid)
-		)
-	)
-	(wire
-		(pts
 			(xy 124.46 121.92) (xy 133.35 121.92)
 		)
@@
 	(wire
 		(pts
-			(xy 58.42 48.26) (xy 85.09 48.26)
-		)
-		(stroke
-			(width 0)
-			(type solid)
-		)
-	)
-	(wire
-		(pts
 			(xy 142.24 52.07) (xy 139.7 52.07)
 		)
@@
 	(wire
 		(pts
+			(xy 60.96 50.8) (xy 60.96 63.5)
+		)
+		(stroke
+			(width 0)
+			(type solid)
+		)
+	)
+	(wire
+		(pts
 			(xy 107.95 33.02) (xy 107.95 35.56)
 		)
@@
 	(wire
 		(pts
+			(xy 58.42 48.26) (xy 85.09 48.26)
+		)
+		(stroke
+			(width 0)
+			(type solid)
+		)
+	)
+	(wire
+		(pts
 			(xy 274.32 41.91) (xy 274.32 43.18)
 		)
@@
 	(wire
 		(pts
-			(xy 60.96 68.58) (xy 60.96 80.01)
-		)
-		(stroke
-			(width 0)
-			(type solid)
-		)
-	)
-	(wire
-		(pts
 			(xy 58.42 53.34) (xy 85.09 53.34)
 		)
@@
 		)
 	)
+	(label "WP"
+		(at 91.44 180.34 0)
+		(effects
+			(font
+				(size 1.27 1.27)
+			)
+			(justify left bottom)
+		)
+	)
 	(label "GPIO2{slash}SDA1"
 		(at 81.28 124.46 180)
@@
 	(symbol
 		(lib_id "Connector_Generic:Conn_02x20_Odd_Even")
-		(at 53.34 50.8 0)
-		(mirror y)
+		(at 50.8 50.8 0)
 		(unit 1)
 		(body_style 1)
@@
 			)
 		)
-		(property "Footprint" "custom:Samtec_HLE-120-02-xxx-DV-BE_2x20_P2.54mm_Horizontal"
-			(at 176.53 74.93 0)
+		(property "Footprint" "Connector_PinSocket_2.54mm:PinSocket_2x20_P2.54mm_Vertical"
+			(at -72.39 74.93 0)
 			(hide yes)
 			(show_name no)
@@
 		)
 		(property "Datasheet" ""
-			(at 176.53 74.93 0)
+			(at -72.39 74.93 0)
 			(hide yes)
 			(show_name no)
@@
 		)
 		(property "Description" "Generic connector, double row, 02x20, odd/even pin numbering scheme (row 1 odd numbers, row 2 even numbers), script generated (kicad-library-utils/schlib/autogen/connector/)"
-			(at 53.34 50.8 0)
+			(at 50.8 50.8 0)
 			(hide yes)
 			(show_name no)
@@
 		)
 		(property "MPN" "HLE-120-02-F-DV-BE"
-			(at 53.34 50.8 0)
+			(at 50.8 50.8 0)
 			(hide yes)
 			(show_name no)
@@
 		)
 		(property "Voltage Rating" ""
-			(at 53.34 50.8 0)
+			(at 50.8 50.8 0)
 			(hide yes)
 			(show_name no)
@@
 			)
 		)
-		(property "MPN" "SM04B-SRSS-TB"
+		(property "MPN" "BM04B-SRSS-TB"
 			(at 217.17 113.03 0)
 			(hide yes)
@@
 			)
 		)
-		(property "MPN" "S4B-PH-SM4-TB"
+		(property "MPN" "B5B-PH-SM4-TB"
 			(at 186.69 113.03 0)
 			(hide yes)
