File: devices/rpi-uHAT/rpi-uHAT.kicad_pcb (KiCad board)
At the start: 2 copper layers, 65 x 30.5 mm, 26 parts, among them J1 GPIO, J2 JST PH, J3 JST SH, J6 PC FAN HEADER, U1 CAT24C256, U2 AP2112K-3.3, U3 EMC2101-x-ACZL, U4 TCA9406DC

Commit message: Finsihes version A.0 of the BLE sensor
Parts:
- added C10: 100u, Capacitor_SMD:C_1206_3216Metric, F.Cu at (105.6, 88.3)
- added C7: 100n, Capacitor_SMD:C_0603_1608Metric, F.Cu at (105.0, 81.0)
- added C8: 33n, Capacitor_SMD:C_0603_1608Metric, F.Cu at (105.0, 86.4)
- added C9: 4u7, Capacitor_SMD:C_0805_2012Metric, F.Cu at (105.0, 90.5)
- added Q1: MMBT3904, Package_TO_SOT_SMD:SOT-23, F.Cu at (112.8, 86.1)
- added Q2: DMG2305UX, Package_TO_SOT_SMD:SOT-23, F.Cu at (105.0, 83.7)
- added R7: 100k, Resistor_SMD:R_0603_1608Metric, F.Cu at (107.5, 83.7)
- added R8: 500m, Resistor_SMD:R_0603_1608Metric, F.Cu at (108.7, 89.6)
- J2: footprint custom:JST_PH_S4B-PH-SM4-TB_1x04-1MP_P2.00mm_Horizontal -> Connector_JST:JST_PH_B5B-PH-SM4-TB_1x05-1MP_P2.00mm_Vertical
- J3: footprint Connector_JST:JST_SH_SM04B-SRSS-TB_1x04-1MP_P1.00mm_Horizontal -> Connector_JST:JST_SH_BM04B-SRSS-TB_1x04-1MP_P1.00mm_Vertical
- U3: value EMC2101-x-ACZL -> EMC2101-ACZL
- moved C3 6.33 mm to (125.3, 97.8), turned to 0 degrees
- moved J3 4.70 mm to (154.1, 92.3), turned to 180 degrees
- moved C2 4.31 mm to (125.3, 92.0), turned to 0 degrees
- moved J2 4.11 mm to (140.5, 92.5)
- moved U2 3.45 mm to (125.3, 94.9), turned to 90 degrees
- moved C5 2.83 mm to (121.6, 82.3)
- moved C6 2.83 mm to (121.6, 89.8)
- moved R3 2.83 mm to (124.2, 87.6)
- moved R4 2.83 mm to (124.2, 84.6)
- moved R5 2.83 mm to (118.9, 88.2)
- moved R6 2.83 mm to (118.9, 84.1)
- moved U3 2.83 mm to (116.4, 86.1)
- moved U4 2.83 mm to (121.6, 86.1)
- moved C4 2.52 mm to (114.2, 90.0)
Connections:
- J2 pad 2: +3V3 -> +5V_RPI
- J2 pad 3: /SDA -> +3V3
- J2 pad 4: /SCL -> /SDA
- J3 pad MP: +3V3 -> unconnected-(J3-MountPin-PadMP)
- J6 pad 2: +5V_RPI -> +5V_FAN
- U3 pad 2: unconnected-(U3-DP-Pad2) -> /DP
- U3 pad 3: unconnected-(U3-DN-Pad3) -> /DN
Routing:
- net /SDA: track 68.6 -> 53.9 mm
- net /SCL: track 62.6 -> 49.2 mm
- net +3V3: track 57.8 -> 69.7 mm
- net /DP: track 0.00 -> 9.57 mm, vias 0 -> 2
- net /SS_G: track 0.00 -> 7.14 mm
- net /DN: track 0.00 -> 6.44 mm, vias 0 -> 2
- net +3V3_RPI: track 139.1 -> 134.0 mm
- net /FAN: track 8.36 -> 11.2 mm
- net /TACH: track 17.3 -> 20.1 mm
- net Net-(C10-Pad2): track 0.00 -> 1.82 mm
- net /EN: track 16.2 -> 15.1 mm
- net /GPIO2/SDA1: track 25.8 -> 24.7 mm
- net /GPIO3/SCL1: track 18.5 -> 17.7 mm
- net GND: track 35.1 -> 36.0 mm, vias 37 -> 40
- added copper zone on F.Cu, net +5V_FAN

Commit message: Tweeks on RPI board
Parts:
- added kibuzzard-6A731D1D: G***, kibuzzard-6A731D1D, B.Cu at (124.2, 88.0)
- J1: footprint custom:Samtec_HLE-120-02-xxx-DV-BE_2x20_P2.54mm_Horizontal -> Connector_PinSocket_2.54mm:PinSocket_2x20_P2.54mm_Vertical; moved to B.Cu
- moved J1 24.2 mm to (108.4, 74.8), turned to -90 degrees
- moved REF** 18.5 mm to (138.7, 87.5)
- moved C2 0.24 mm to (125.3, 91.8)
- moved C3 0.16 mm to (125.3, 98.0)
Connections:
- net Net-(JP1-A) renamed /WP
- J1 pad 1: +5V_RPI -> +3V3_RPI
- J1 pad 10: GND -> /GPIO15/RXD0
- J1 pad 11: /GPIO18/PCM.CLK -> /GPIO17
- J1 pad 12: /GPIO17 -> /GPIO18/PCM.CLK
- J1 pad 13: GND -> /GPIO27
- J1 pad 14: /GPIO27 -> GND
- J1 pad 15: /GPIO23 -> /GPIO22
- J1 pad 16: /GPIO22 -> /GPIO23
- J1 pad 17: /GPIO24 -> +3V3_RPI
- J1 pad 18: +3V3_RPI -> /GPIO24
- J1 pad 19: GND -> /GPIO10/SPI0.MOSI
- J1 pad 2: +3V3_RPI -> +5V_RPI
- J1 pad 20: /GPIO10/SPI0.MOSI -> GND
- J1 pad 21: /GPIO25 -> /GPIO9/SPI0.MISO
- J1 pad 22: /GPIO9/SPI0.MISO -> /GPIO25
- J1 pad 23: /GPIO8/SPI0.CE0 -> /GPIO11/SPI0.SCLK
- J1 pad 24: /GPIO11/SPI0.SCLK -> /GPIO8/SPI0.CE0
- J1 pad 25: /GPIO7/SPI0.CE1 -> GND
- J1 pad 26: GND -> /GPIO7/SPI0.CE1
- J1 pad 27: /ID_SCL -> /ID_SDA
- J1 pad 28: /ID_SDA -> /ID_SCL
- J1 pad 29: GND -> /GPIO5
- J1 pad 3: +5V_RPI -> /GPIO2/SDA1
- J1 pad 30: /GPIO5 -> GND
- J1 pad 31: /GPIO12/PWM0 -> /GPIO6
- J1 pad 32: /GPIO6 -> /GPIO12/PWM0
- J1 pad 33: GND -> /GPIO13/PWM1
- J1 pad 34: /GPIO13/PWM1 -> GND
- J1 pad 35: /GPIO16 -> /GPIO19/PCM.FS
- J1 pad 36: /GPIO19/PCM.FS -> /GPIO16
- J1 pad 37: /GPIO20/PCM.DIN -> /GPIO26
- J1 pad 38: /GPIO26 -> /GPIO20/PCM.DIN
- J1 pad 39: /GPIO21/PCM.DOUT -> GND
- J1 pad 4: /GPIO2/SDA1 -> +5V_RPI
- J1 pad 40: GND -> /GPIO21/PCM.DOUT
- J1 pad 5: GND -> /GPIO3/SCL1
- J1 pad 6: /GPIO3/SCL1 -> GND
- J1 pad 7: /GPIO14/TXD0 -> /EN
- J1 pad 8: /EN -> /GPIO14/TXD0
- J1 pad 9: /GPIO15/RXD0 -> GND
Routing:
- net +3V3_RPI: track 134.0 -> 103.4 mm, vias 2 -> 0
- net GND: track 36.0 -> 19.5 mm, vias 40 -> 25
- net /ID_SCL: track 29.7 -> 31.3 mm
- net /GPIO3/SCL1: track 17.7 -> 19.2 mm
- net /GPIO2/SDA1: track 24.7 -> 23.3 mm
- net /EN: track 15.1 -> 16.2 mm
Other:
- board size 65 x 30.5 mm -> 65 x 30 mm
