File: devices/BLE_environmental-sensor/BLE_environmental-sensor.kicad_sch (KiCad schematic)
At the start: 16 parts, among them J1 Conn_02x05_Odd_Even, Q1 Q_PMOS_GSD, U1 BGM220SC12WGA2R, U2 SHT4x, U3 STCC4, U4 LPS22DF, U5 TPS61291DVR, Y1 32.768kHz

Commit message: [wip] More stuff
Parts:
- BT1: footprint Battery:BatteryHolder_Multicomp_BC-2001_1x2032 -> custom:BatteryHolder_MPD_BK-912
Connections:
- net PTI_DATA: now also U1.32 (PC04); no longer U1.26 (PD01/XTAL1)
- net PTI_FRAME: now also U1.33 (PC05); no longer U1.27 (PD00/XTAL0)
Changed lines of the file:
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@@
 		(pin "37"
 		)
+		(pin "32"
+		)
 		(pin "26"
 		)
-		(pin "26"
-		)
 		(pin "31"
 		)
@@
 		(pin "25"
 		)
-		(pin "27"
+		(pin "33"
 		)
 		(pin "39"
@@
 			)
 		)
-		(property "Footprint" "Battery:BatteryHolder_Multicomp_BC-2001_1x2032"
+		(property "Footprint" "custom:BatteryHolder_MPD_BK-912"
 			(at 185.42 27.686 90)
 			(hide yes)
