File: devices/USB_LED_Ring/USB_LED_Ring.kicad_sch (KiCad schematic)
At the start: 76 parts, among them J1 JST SH 3 Vert, J2 USB_B_Micro, J3 JST SH 3 Vert, J4 .100, U1 TPS923610, U2 TLV75733PDBV, U3 RP2354A, U4 TPS25947xx, Y1 ABM8-272-T3

Commit message: Finsihes version A.0 of the BLE sensor
Parts:
- C1: MPN (none) -> GRM21BZ71H475ME15
- C10, C11, C12: MPN GRM155Z71A225KE01D -> GRM188Z71A475ME15D
- C13, C14, C15, C16, C17, C18, C19, C2, C8, C9: MPN CL05B104KP5NNNC -> CL05B104KO5NNN
- C20: MPN CL10B225KP8NNNC -> GRM21BZ71H475ME15
- C21: MPN CL05B104KP5NNNC -> GRM1555C1H102JA01D
- C3, C5: MPN CL10B225KP8NNNC -> CL21B225KBYNNWE
- C4: value 1u -> 2u2; footprint Capacitor_SMD:C_0603_1608Metric -> Capacitor_SMD:C_0805_2012Metric; MPN (none) -> CL21B225KBYNNWE; Voltage Rating 25V -> (none)
- D1, D10, D11, D12, D13, D14, D15, D16, D17, D18, D19, D2, D20, D21, D22, D23, D24, D3, D4, D5, D6, D7, D8, D9: MPN (none) -> 158301250
- J1, J3: MPN (none) -> BM03B-SRSS-TB
- L2: MPN (none) -> AOTA-B252010S3R3MT
- R1: MPN (none) -> CPF0603B2R55E1
- R10: MPN (none) -> RC0402FR-07130KL
- R11, R9: MPN (none) -> RC0402FR-0747KL
- R2: MPN (none) -> KDV06FR100ET
- R7: MPN (none) -> RC0402FR-076K8L
- R8: MPN (none) -> RC0402FR-07430KL
- TP1, TP2, TP3, TP4, TP5, TP6: MPN (none) -> RCUCTE
- U1: MPN (none) -> TPS923610DRLR
