File: devices/tunnel-IR-barrier/tunnel-IR-barrier.kicad_pcb (KiCad board)
At the start: 2 copper layers, 10 x 45.5 mm, 23 parts, among them J1 JST SH 5, J2 JST SH 5, J4 JST SH 2, Q1 RE1C002UN, Q2 RE1C002UN, Q3 RE1C002UN, Q4 RE1C001ZP, U1 ATtiny204-SS, U2 GP2S700HCP, U3 GP2S700HCP, U4 GP2S700HCP

Commit message: Finsihes version A.0 of the BLE sensor
Parts:
- J4: footprint Connector_JST:JST_SH_BM03B-SRSS-TB_1x03-1MP_P1.00mm_Vertical -> Connector_JST:JST_SH_SM03B-SRSS-TB_1x03-1MP_P1.00mm_Horizontal; moved to F.Cu
- Q1, Q2, Q3, Q4: footprint Package_TO_SOT_SMD:SOT-416 -> custom:SOT-416
- moved J4 19.6 mm to (150.5, 95.0), turned to 0 degrees
- moved J1 4.60 mm to (150.5, 87.5)
- moved J2 4.60 mm to (150.5, 95.5)
Connections:
- J4 pad MP: GND -> unconnected-(J4-MountPin-PadMP)_1
Routing:
- net /UDPI/~{RST}: track 4.43 -> 16.7 mm, vias 1 -> 0
- net GND: track 3.67 -> 15.3 mm, vias 5 -> 6
- net +3V3: track 70.0 -> 78.6 mm, vias 5 -> 3
- net /DOUT: track 11.3 -> 14.7 mm
- net /DIN: track 5.05 -> 8.01 mm
- net /CLK: track 12.0 -> 13.3 mm
- net /~{SS} : track 11.9 -> 12.9 mm
Other:
- board size 10 x 45.5 mm -> 10 x 50 mm
