File: devices/tunnel-IR-barrier/tunnel-IR-barrier.kicad_sch (KiCad schematic)
At the start: 17 parts, among them J1 JST SH 5, J2 JST SH 5, J4 JST SH 2, Q1 RE1C002UN, Q2 RE1C002UN, Q3 RE1C002UN, Q4 RE1C001ZP, U1 ATtiny204-SS, U2 GP2S700HCP, U3 GP2S700HCP, U4 GP2S700HCP

Commit message: Finsihes version A.0 of the BLE sensor
Parts:
- J4: footprint Connector_JST:JST_SH_BM03B-SRSS-TB_1x03-1MP_P1.00mm_Vertical -> Connector_JST:JST_SH_SM03B-SRSS-TB_1x03-1MP_P1.00mm_Horizontal
- Q1, Q2, Q3, Q4: footprint Package_TO_SOT_SMD:SOT-416 -> custom:SOT-416
Connections:
- net GND: no longer J4.MP (MountPin)
- no-connect marks 2 -> 3
Changed lines of the file:
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@@
 	)
 	(junction
-		(at 224.79 134.62)
-		(diameter 0)
-		(color 0 0 0 0)
-	)
-	(junction
 		(at 224.79 38.1)
 		(diameter 0)
@@
 		(at 148.59 55.88)
 	)
-	(wire
-		(pts
-			(xy 72.39 39.37) (xy 72.39 86.36)
-		)
-		(stroke
-			(width 0)
-			(type default)
-		)
+	(no_connect
+		(at 231.14 142.24)
 	)
 	(wire
 		(pts
-			(xy 224.79 144.78) (xy 231.14 144.78)
+			(xy 72.39 39.37) (xy 72.39 86.36)
 		)
 		(stroke
@@
 	(wire
 		(pts
-			(xy 231.14 144.78) (xy 231.14 142.24)
-		)
-		(stroke
-			(width 0)
-			(type default)
-		)
-	)
-	(wire
-		(pts
 			(xy 224.79 125.73) (xy 224.79 132.08)
 		)
@@
 	(wire
 		(pts
-			(xy 226.06 134.62) (xy 224.79 134.62)
-		)
-		(stroke
-			(width 0)
-			(type default)
-		)
-	)
-	(wire
-		(pts
 			(xy 26.67 99.06) (xy 29.21 99.06)
 		)
@@
 	(wire
 		(pts
-			(xy 224.79 134.62) (xy 222.25 134.62)
+			(xy 222.25 134.62) (xy 226.06 134.62)
 		)
 		(stroke
@@
 	(wire
 		(pts
-			(xy 224.79 134.62) (xy 224.79 144.78)
-		)
-		(stroke
-			(width 0)
-			(type default)
-		)
-	)
-	(wire
-		(pts
 			(xy 57.15 138.43) (xy 57.15 142.24)
 		)
@@
 			)
 		)
-		(property "Footprint" "Package_TO_SOT_SMD:SOT-416"
+		(property "Footprint" "custom:SOT-416"
 			(at 39.37 49.53 0)
 			(hide yes)
@@
 			)
 		)
-		(property "Footprint" "Package_TO_SOT_SMD:SOT-416"
+		(property "Footprint" "custom:SOT-416"
 			(at 39.37 96.52 0)
 			(hide yes)
@@
 			)
 		)
-		(property "Footprint" "Connector_JST:JST_SH_BM03B-SRSS-TB_1x03-1MP_P1.00mm_Vertical"
+		(property "Footprint" "Connector_JST:JST_SH_SM03B-SRSS-TB_1x03-1MP_P1.00mm_Horizontal"
 			(at 231.14 134.62 0)
 			(hide yes)
@@
 			)
 		)
-		(property "Footprint" "Package_TO_SOT_SMD:SOT-416"
+		(property "Footprint" "custom:SOT-416"
 			(at 77.47 36.83 0)
 			(hide yes)
@@
 			)
 		)
-		(property "Footprint" "Package_TO_SOT_SMD:SOT-416"
+		(property "Footprint" "custom:SOT-416"
 			(at 39.37 148.59 0)
 			(hide yes)
